File: hardware/rev1/delta-m0/delta-m0.kicad_pcb (KiCad board)
At the start: 2 copper layers, 44.5 x 82 mm, 52 parts, among them J1 Battery, J2 ProgrammingHeader, SW1 PowerSwitch, SW10 SW_Push, SW11 SW_Push, SW12 SW_Push, SW13 SW_Push, SW14 SW_Push, SW15 SW_Push, SW16 SW_Push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

Commit message: Update Kicad PCB
Other:
- board text added: "JLCJLCJLCJLC"
